File: uav_router.brd (EAGLE design)
At the start: 100 x 80 mm, 15 parts

Commit message: Adding MCLR
Connections:
- net N$1 renamed MCLR
Changed lines of the file:
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@@
 <wire x1="64.77" y1="7.62" x2="62.23" y2="7.62" width="0.4064" layer="1"/>
 </signal>
-<signal name="N$1">
+<signal name="MCLR">
 <contactref element="U$1" pad="1"/>
 <contactref element="R1" pad="P$1"/>

Commit message: Adding ICSP programming interface
Parts:
- added U$2: PIC-ICSPPOLAR_LOCK, SparkFun-Connectors:MOLEX-1X6_LOCK
Connections:
- new net PGC: U$1.27, U$2.2
- new net PGD: U$1.28, U$2.3
- new net VCC_NC: U$2.5
- net GND: now also U$2.4
- net MCLR: now also U$2.6
Changed lines of the file:
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@@
 <element name="R5" library="SparkFun-Resistors" package="AXIAL-0.3-KIT" value="" x="2.54" y="36.83" rot="R90"/>
 <element name="PWR" library="SparkFun-LED" package="LED5MM" value="" x="12.7" y="49.53" rot="R180"/>
+<element name="U$2" library="SparkFun-Connectors" package="MOLEX-1X6_LOCK" value="PIC-ICSPPOLAR_LOCK" x="2.54" y="-6.35"/>
 </elements>
 <signals>
@@
 <wire x1="62.23" y1="19.05" x2="66.04" y2="15.24" width="0.4064" layer="1"/>
 <wire x1="66.04" y1="15.24" x2="66.04" y2="1.27" width="0.4064" layer="1"/>
+<contactref element="U$2" pad="4"/>
+<wire x1="2.54" y1="1.27" x2="10.16" y2="-6.604" width="0" layer="19" extent="1-1"/>
 </signal>
 <signal name="5V">
@@
 <contactref element="R1" pad="P$1"/>
 <wire x1="16.51" y1="12.7" x2="12.7" y2="12.7" width="0.4064" layer="1"/>
+<contactref element="U$2" pad="6"/>
+<wire x1="15.24" y1="-6.604" x2="16.51" y2="12.7" width="0" layer="19" extent="1-1"/>
 </signal>
 <signal name="OSC2">
@@
 <wire x1="2.54" y1="40.64" x2="11.43" y2="49.53" width="0.4064" layer="1"/>
 </signal>
+<signal name="VCC_NC">
+<contactref element="U$2" pad="5"/>
+</signal>
+<signal name="PGD">
+<contactref element="U$2" pad="3"/>
+<contactref element="U$1" pad="28"/>
+<wire x1="7.62" y1="-6.35" x2="16.51" y2="20.32" width="0" layer="19" extent="1-1"/>
+</signal>
+<signal name="PGC">
+<contactref element="U$2" pad="2"/>
+<contactref element="U$1" pad="27"/>
+<wire x1="5.08" y1="-6.604" x2="19.05" y2="20.32" width="0" layer="19" extent="1-1"/>
+</signal>
 </signals>

Commit message: Routed ICSP programming interface
Parts:
- removed U$2: PIC-ICSPPOLAR_LOCK, SparkFun-Connectors:MOLEX-1X6_LOCK
- added ISCP: (no value), SparkFun-Connectors:MOLEX-1X6_LOCK
Connections:
- net GND: now also ISCP.4; no longer U$2.4
- net MCLR: now also ISCP.6; no longer U$2.6
- net PGC: now also ISCP.2; no longer U$2.2
- net PGD: now also ISCP.3; no longer U$2.3
- net VCC_NC: now also ISCP.5; no longer U$2.5
Routing:
- net GND: track 456.9 -> 476.7 mm
- net PGD: track 0.00 -> 16.8 mm
- net PGC: track 0.00 -> 16.6 mm
- net MCLR: track 3.81 -> 9.69 mm
Changed lines of the file:
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@@
 <element name="R5" library="SparkFun-Resistors" package="AXIAL-0.3-KIT" value="" x="2.54" y="36.83" rot="R90"/>
 <element name="PWR" library="SparkFun-LED" package="LED5MM" value="" x="12.7" y="49.53" rot="R180"/>
-<element name="U$2" library="SparkFun-Connectors" package="MOLEX-1X6_LOCK" value="PIC-ICSPPOLAR_LOCK" x="2.54" y="-6.35"/>
+<element name="ISCP" library="SparkFun-Connectors" package="MOLEX-1X6_LOCK" value="" x="26.67" y="6.35" rot="R180"/>
 </elements>
 <signals>
@@
 <wire x1="62.23" y1="19.05" x2="66.04" y2="15.24" width="0.4064" layer="1"/>
 <wire x1="66.04" y1="15.24" x2="66.04" y2="1.27" width="0.4064" layer="1"/>
-<contactref element="U$2" pad="4"/>
-<wire x1="2.54" y1="1.27" x2="10.16" y2="-6.604" width="0" layer="19" extent="1-1"/>
+<contactref element="ISCP" pad="4"/>
+<wire x1="19.05" y1="6.604" x2="19.05" y2="7.62" width="0.4064" layer="16"/>
+<wire x1="19.05" y1="7.62" x2="20.32" y2="8.89" width="0.4064" layer="16"/>
+<wire x1="20.32" y1="8.89" x2="33.02" y2="8.89" width="0.4064" layer="16"/>
+<wire x1="33.02" y1="8.89" x2="34.29" y2="10.16" width="0.4064" layer="16"/>
+<wire x1="34.29" y1="10.16" x2="34.29" y2="12.7" width="0.4064" layer="16"/>
 </signal>
 <signal name="5V">
@@
 <contactref element="U$1" pad="1"/>
 <contactref element="R1" pad="P$1"/>
-<wire x1="16.51" y1="12.7" x2="12.7" y2="12.7" width="0.4064" layer="1"/>
-<contactref element="U$2" pad="6"/>
-<wire x1="15.24" y1="-6.604" x2="16.51" y2="12.7" width="0" layer="19" extent="1-1"/>
+<contactref element="ISCP" pad="6"/>
+<wire x1="13.97" y1="6.604" x2="13.97" y2="11.43" width="0.4064" layer="1"/>
+<wire x1="13.97" y1="11.43" x2="12.7" y2="12.7" width="0.4064" layer="1"/>
+<wire x1="16.51" y1="12.7" x2="15.24" y2="12.7" width="0.4064" layer="1"/>
+<wire x1="15.24" y1="12.7" x2="13.97" y2="11.43" width="0.4064" layer="1"/>
 </signal>
 <signal name="OSC2">
@@
 </signal>
 <signal name="VCC_NC">
-<contactref element="U$2" pad="5"/>
+<contactref element="ISCP" pad="5"/>
 </signal>
 <signal name="PGD">
-<contactref element="U$2" pad="3"/>
+<contactref element="ISCP" pad="3"/>
 <contactref element="U$1" pad="28"/>
-<wire x1="7.62" y1="-6.35" x2="16.51" y2="20.32" width="0" layer="19" extent="1-1"/>
+<wire x1="16.51" y1="20.32" x2="16.51" y2="15.24" width="0.4064" layer="1"/>
+<wire x1="16.51" y1="15.24" x2="17.78" y2="13.97" width="0.4064" layer="1"/>
+<wire x1="17.78" y1="13.97" x2="17.78" y2="10.16" width="0.4064" layer="1"/>
+<wire x1="17.78" y1="10.16" x2="19.05" y2="8.89" width="0.4064" layer="1"/>
+<wire x1="19.05" y1="8.89" x2="20.32" y2="8.89" width="0.4064" layer="1"/>
+<wire x1="20.32" y1="8.89" x2="21.59" y2="7.62" width="0.4064" layer="1"/>
+<wire x1="21.59" y1="7.62" x2="21.59" y2="6.35" width="0.4064" layer="1"/>
 </signal>
 <signal name="PGC">
-<contactref element="U$2" pad="2"/>
+<contactref element="ISCP" pad="2"/>
 <contactref element="U$1" pad="27"/>
-<wire x1="5.08" y1="-6.604" x2="19.05" y2="20.32" width="0" layer="19" extent="1-1"/>
+<wire x1="19.05" y1="20.32" x2="19.05" y2="15.24" width="0.4064" layer="1"/>
+<wire x1="19.05" y1="15.24" x2="20.32" y2="13.97" width="0.4064" layer="1"/>
+<wire x1="20.32" y1="13.97" x2="20.32" y2="10.16" width="0.4064" layer="1"/>
+<wire x1="20.32" y1="10.16" x2="21.59" y2="8.89" width="0.4064" layer="1"/>
+<wire x1="21.59" y1="8.89" x2="22.86" y2="8.89" width="0.4064" layer="1"/>
+<wire x1="22.86" y1="8.89" x2="24.13" y2="7.62" width="0.4064" layer="1"/>
+<wire x1="24.13" y1="7.62" x2="24.13" y2="6.604" width="0.4064" layer="1"/>
 </signal>
 </signals>
