File: uav_controller.sch (EAGLE design)
At the start: 19 parts, among them IC1 PIC16F877SO, U3 LCD-16X28X2

Commit message: Adding board-interconnect https://www.sparkfun.com/products/10651 https://www.sparkfun.com/products/10647 https://www.sparkfun.com/products/10877
Parts:
- added JP6, JP7: (no value), SparkFun-Connectors:M03X2
- added RANGE_VOLTAGE: (no value), SparkFun-Connectors:M03PTH
- JP5: device SparkFun-Connectors:M03PTH -> SparkFun-Connectors:M03X2
- OSC: value 8Mhz -> 20Mhz
- renumbered IC1 to FLIGHTCTRL
Connections:
- removed net N$11: FLIGHTCTRL.TX/RC6
- removed net N$12: FLIGHTCTRL.RX/RC7
- new net N$15: JP5.6, JP6.6, JP7.6
- new net RX: FLIGHTCTRL.RX/RC7, JP5.2, JP6.2, JP7.2
- new net TX: FLIGHTCTRL.TX/RC6, JP5.4, JP6.4, JP7.4
- net 3.3V: now also JP6.1, JP7.1, RANGE_VOLTAGE.1
- net 5V: now also JP6.3, JP7.3, RANGE_VOLTAGE.3
- net GND: now also JP5.5, JP6.5, JP7.5
- net N$17: now also RANGE_VOLTAGE.2; no longer JP5.2

Commit message: Adding ICSP
Parts:
- added R2, R3: (no value), SparkFun-Resistors:RESISTORKIT
- added U$1: PIC-ICSPPOLAR_LOCK, SparkFun-Connectors:PIC-ICSPPOLAR_LOCK
Connections:
- removed net N$1: FLIGHTCTRL.!MCLR/THV, R1.1
- new net MCLR: FLIGHTCTRL.!MCLR/THV, R1.1, U$1.VPP
- new net PGC: FLIGHTCTRL.PGC/RB6, R3.1, U$1.PGC
- new net PGD: FLIGHTCTRL.PGD/RB7, R2.1, U$1.PGD
- new net VCC_NC: U$1.VCC
- net GND: now also U$1.GND
- net RWD3: now also R3.2; no longer FLIGHTCTRL.PGC/RB6
- net RWD4: now also R2.2; no longer FLIGHTCTRL.PGD/RB7
Other:
- moved on the sheet: R1
Changed lines of the file:
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@@
 <part name="SUPPLY8" library="SparkFun-Aesthetics" deviceset="5V" device=""/>
 <part name="GND9" library="SparkFun-Aesthetics" deviceset="GND" device=""/>
+<part name="U$1" library="SparkFun-Connectors" deviceset="PIC-ICSP" device="POLAR_LOCK"/>
+<part name="GND10" library="SparkFun-Aesthetics" deviceset="GND" device=""/>
+<part name="R2" library="SparkFun-Resistors" deviceset="RESISTOR" device="KIT"/>
+<part name="R3" library="SparkFun-Resistors" deviceset="RESISTOR" device="KIT"/>
 </parts>
 <sheets>
@@
 <instance part="SUPPLY5" gate="1" x="43.18" y="167.64"/>
 <instance part="SUPPLY6" gate="1" x="241.3" y="142.24"/>
-<instance part="R1" gate="G$1" x="157.48" y="162.56" rot="R90"/>
+<instance part="R1" gate="G$1" x="162.56" y="162.56" rot="R90"/>
 <instance part="HBRIDGE-FRONT" gate="G$1" x="259.08" y="129.54"/>
 <instance part="HBRIDGE-REAR" gate="G$1" x="259.08" y="99.06"/>
@@
 <instance part="SUPPLY8" gate="G$1" x="162.56" y="223.52"/>
 <instance part="GND9" gate="1" x="165.1" y="185.42"/>
+<instance part="U$1" gate="G$1" x="106.68" y="50.8"/>
+<instance part="GND10" gate="1" x="134.62" y="35.56"/>
+<instance part="R2" gate="G$1" x="256.54" y="172.72"/>
+<instance part="R3" gate="G$1" x="256.54" y="167.64"/>
 </instances>
 <busses>
@@
 <wire x1="223.52" y1="180.34" x2="152.4" y2="180.34" width="0.762" layer="92"/>
 <wire x1="152.4" y1="180.34" x2="149.86" y2="177.8" width="0.762" layer="92"/>
-<wire x1="149.86" y1="177.8" x2="149.86" y2="83.82" width="0.762" layer="92"/>
+<wire x1="149.86" y1="177.8" x2="149.86" y2="30.48" width="0.762" layer="92"/>
 </segment>
 </bus>
@@
 <junction x="165.1" y="203.2"/>
 </segment>
+<segment>
+<pinref part="U$1" gate="G$1" pin="GND"/>
+<pinref part="GND10" gate="1" pin="GND"/>
+<wire x1="114.3" y1="50.8" x2="134.62" y2="50.8" width="0.1524" layer="91"/>
+<wire x1="134.62" y1="50.8" x2="134.62" y2="38.1" width="0.1524" layer="91"/>
+<label x="116.84" y="50.8" size="1.778" layer="95"/>
+</segment>
 </net>
 <net name="3.3V" class="0">
@@
 <junction x="185.42" y="167.64"/>
 <pinref part="R1" gate="G$1" pin="2"/>
-<wire x1="157.48" y1="167.64" x2="185.42" y2="167.64" width="0.1524" layer="91"/>
+<wire x1="162.56" y1="167.64" x2="185.42" y2="167.64" width="0.1524" layer="91"/>
 </segment>
 <segment>
@@
 <net name="RWD3" class="0">
 <segment>
-<pinref part="FLIGHTCTRL" gate="G$1" pin="PGC/RB6"/>
-<wire x1="208.28" y1="152.4" x2="220.98" y2="152.4" width="0.1524" layer="91"/>
-<wire x1="220.98" y1="152.4" x2="223.52" y2="154.94" width="0.1524" layer="91"/>
-<label x="210.82" y="152.4" size="1.778" layer="95"/>
-</segment>
-<segment>
 <pinref part="HBRIDGE-REAR" gate="G$1" pin="IN3"/>
 <wire x1="274.32" y1="101.6" x2="297.18" y2="101.6" width="0.1524" layer="91"/>
@@
 <wire x1="297.18" y1="101.6" x2="299.72" y2="104.14" width="0.1524" layer="91"/>
 </segment>
+<segment>
+<pinref part="R3" gate="G$1" pin="2"/>
+<wire x1="261.62" y1="167.64" x2="297.18" y2="167.64" width="0.1524" layer="91"/>
+<wire x1="297.18" y1="167.64" x2="299.72" y2="170.18" width="0.1524" layer="91"/>
+<label x="287.02" y="167.64" size="1.778" layer="95"/>
+</segment>
 </net>
 <net name="RWD4" class="0">
-<segment>
-<pinref part="FLIGHTCTRL" gate="G$1" pin="PGD/RB7"/>
-<wire x1="208.28" y1="154.94" x2="220.98" y2="154.94" width="0.1524" layer="91"/>
-<wire x1="220.98" y1="154.94" x2="223.52" y2="157.48" width="0.1524" layer="91"/>
-<label x="210.82" y="154.94" size="1.778" layer="95"/>
-</segment>
 <segment>
 <pinref part="HBRIDGE-REAR" gate="G$1" pin="IN4"/>
@@
 <wire x1="297.18" y1="99.06" x2="299.72" y2="101.6" width="0.1524" layer="91"/>
 </segment>
-</net>
-<net name="N$1" class="0">
+<segment>
+<pinref part="R2" gate="G$1" pin="2"/>
+<wire x1="261.62" y1="172.72" x2="297.18" y2="172.72" width="0.1524" layer="91"/>
+<wire x1="297.18" y1="172.72" x2="299.72" y2="175.26" width="0.1524" layer="91"/>
+<label x="287.02" y="172.72" size="1.778" layer="95"/>
+</segment>
+</net>
+<net name="MCLR" class="0">
 <segment>
 <pinref part="FLIGHTCTRL" gate="G$1" pin="!MCLR/THV"/>
 <pinref part="R1" gate="G$1" pin="1"/>
-<wire x1="165.1" y1="157.48" x2="157.48" y2="157.48" width="0.1524" layer="91"/>
+<wire x1="165.1" y1="157.48" x2="162.56" y2="157.48" width="0.1524" layer="91"/>
+<wire x1="162.56" y1="157.48" x2="152.4" y2="157.48" width="0.1524" layer="91"/>
+<wire x1="152.4" y1="157.48" x2="149.86" y2="160.02" width="0.1524" layer="91"/>
+<label x="152.4" y="157.48" size="1.778" layer="95"/>
+</segment>
+<segment>
+<pinref part="U$1" gate="G$1" pin="VPP"/>
+<wire x1="114.3" y1="55.88" x2="147.32" y2="55.88" width="0.1524" layer="91"/>
+<wire x1="147.32" y1="55.88" x2="149.86" y2="58.42" width="0.1524" layer="91"/>
+<label x="116.84" y="55.88" size="1.778" layer="95"/>
 </segment>
 </net>
@@
 </segment>
 </net>
+<net name="VCC_NC" class="0">
+<segment>
+<pinref part="U$1" gate="G$1" pin="VCC"/>
+<wire x1="114.3" y1="53.34" x2="137.16" y2="53.34" width="0.1524" layer="91"/>
+<label x="116.84" y="53.34" size="1.778" layer="95"/>
+</segment>
+</net>
+<net name="PGD" class="0">
+<segment>
+<pinref part="U$1" gate="G$1" pin="PGD"/>
+<wire x1="114.3" y1="48.26" x2="147.32" y2="48.26" width="0.1524" layer="91"/>
+<wire x1="147.32" y1="48.26" x2="149.86" y2="50.8" width="0.1524" layer="91"/>
+<label x="116.84" y="48.26" size="1.778" layer="95"/>
+</segment>
+<segment>
+<pinref part="FLIGHTCTRL" gate="G$1" pin="PGD/RB7"/>
+<wire x1="208.28" y1="154.94" x2="220.98" y2="154.94" width="0.1524" layer="91"/>
+<wire x1="220.98" y1="154.94" x2="223.52" y2="157.48" width="0.1524" layer="91"/>
+<label x="210.82" y="154.94" size="1.778" layer="95"/>
+</segment>
+<segment>
+<pinref part="R2" gate="G$1" pin="1"/>
+<wire x1="251.46" y1="172.72" x2="226.06" y2="172.72" width="0.1524" layer="91"/>
+<wire x1="226.06" y1="172.72" x2="223.52" y2="175.26" width="0.1524" layer="91"/>
+<label x="231.14" y="172.72" size="1.778" layer="95"/>
+</segment>
+</net>
+<net name="PGC" class="0">
+<segment>
+<pinref part="U$1" gate="G$1" pin="PGC"/>
+<wire x1="114.3" y1="45.72" x2="147.32" y2="45.72" width="0.1524" layer="91"/>
+<wire x1="147.32" y1="45.72" x2="149.86" y2="48.26" width="0.1524" layer="91"/>
+<label x="116.84" y="45.72" size="1.778" layer="95"/>
+</segment>
+<segment>
+<pinref part="FLIGHTCTRL" gate="G$1" pin="PGC/RB6"/>
+<wire x1="208.28" y1="152.4" x2="220.98" y2="152.4" width="0.1524" layer="91"/>
+<wire x1="220.98" y1="152.4" x2="223.52" y2="154.94" width="0.1524" layer="91"/>
+<label x="210.82" y="152.4" size="1.778" layer="95"/>
+</segment>
+<segment>
+<pinref part="R3" gate="G$1" pin="1"/>
+<wire x1="251.46" y1="167.64" x2="226.06" y2="167.64" width="0.1524" layer="91"/>
+<wire x1="226.06" y1="167.64" x2="223.52" y2="170.18" width="0.1524" layer="91"/>
+<label x="231.14" y="167.64" size="1.778" layer="95"/>
+</segment>
+</net>

Commit message: Relabeled parts for clarity
Parts:
- CPU: value PIC16F877SO -> '16F877
- renumbered FLIGHTCTRL to CPU, U$1 to ICSP
