File: uav_router.sch (EAGLE design)
At the start: 16 parts

Commit message: Routed ICSP programming interface
Parts:
- renumbered U$2 to ISCP
Changed lines of the file:
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@@
 <part name="R5" library="SparkFun-Resistors" deviceset="RESISTOR" device="KIT"/>
 <part name="PWR" library="SparkFun-LED" deviceset="LED" device="5MM"/>
-<part name="U$2" library="SparkFun-Connectors" deviceset="PIC-ICSP" device="POLAR_LOCK"/>
+<part name="ISCP" library="SparkFun-Connectors" deviceset="PIC-ICSP" device="POLAR_LOCK" value=""/>
 <part name="GND10" library="SparkFun-Aesthetics" deviceset="GND" device=""/>
 </parts>
@@
 <instance part="R5" gate="G$1" x="5.08" y="157.48"/>
 <instance part="PWR" gate="G$1" x="17.78" y="157.48" rot="R270"/>
-<instance part="U$2" gate="G$1" x="-2.54" y="78.74"/>
+<instance part="ISCP" gate="G$1" x="-2.54" y="78.74"/>
 <instance part="GND10" gate="1" x="25.4" y="63.5"/>
 </instances>
@@
 </segment>
 <segment>
-<pinref part="U$2" gate="G$1" pin="GND"/>
+<pinref part="ISCP" gate="G$1" pin="GND"/>
 <pinref part="GND10" gate="1" pin="GND"/>
 <wire x1="5.08" y1="78.74" x2="25.4" y2="78.74" width="0.1524" layer="91"/>
@@
 </segment>
 <segment>
-<pinref part="U$2" gate="G$1" pin="VPP"/>
+<pinref part="ISCP" gate="G$1" pin="VPP"/>
 <wire x1="5.08" y1="83.82" x2="38.1" y2="83.82" width="0.1524" layer="91"/>
 <wire x1="38.1" y1="83.82" x2="40.64" y2="86.36" width="0.1524" layer="91"/>
@@
 <net name="VCC_NC" class="0">
 <segment>
-<pinref part="U$2" gate="G$1" pin="VCC"/>
+<pinref part="ISCP" gate="G$1" pin="VCC"/>
 <wire x1="5.08" y1="81.28" x2="27.94" y2="81.28" width="0.1524" layer="91"/>
 <label x="7.62" y="81.28" size="1.778" layer="95"/>
@@
 <net name="PGD" class="0">
 <segment>
-<pinref part="U$2" gate="G$1" pin="PGD"/>
+<pinref part="ISCP" gate="G$1" pin="PGD"/>
 <wire x1="5.08" y1="76.2" x2="38.1" y2="76.2" width="0.1524" layer="91"/>
 <wire x1="38.1" y1="76.2" x2="40.64" y2="78.74" width="0.1524" layer="91"/>
@@
 <net name="PGC" class="0">
 <segment>
-<pinref part="U$2" gate="G$1" pin="PGC"/>
+<pinref part="ISCP" gate="G$1" pin="PGC"/>
 <wire x1="5.08" y1="73.66" x2="38.1" y2="73.66" width="0.1524" layer="91"/>
 <wire x1="38.1" y1="73.66" x2="40.64" y2="76.2" width="0.1524" layer="91"/>
